Commit message: add inertia

File: my_robot_description/urdf/arm.xacro (robot description, xacro)
@@ -16,4 +16,12 @@
                 <material name="${color}" />
             </visual>
+            <collision>
+                <geometry>
+                    <cylinder radius="${arm_radius}" length="${arm_length}" />
+                </geometry>
+                <origin xyz="${x} ${y} ${z}" />
+            </collision>
+            <xacro:cylinder_inertia m="0.3" r="${arm_radius}" h="${arm_length}"
+                                    o_xyz="${x} ${y} ${z}" o_rpy="0 0 0" />
         </link>
     </xacro:macro>
@@ -27,4 +35,11 @@
             <material name="orange" />
         </visual>
+        <collision>
+            <geometry>
+                <box size="${arm_base_length} ${arm_base_width} ${arm_base_height}" />
+            </geometry>
+        </collision>
+        <xacro:box_inertia m="0.5" x="${arm_base_length}" y="${arm_base_width}" z="${arm_base_height}"
+                           o_xyz="0 0 0" o_rpy="0 0 0" />
     </link>
     <xacro:arms name="forearm" x="0" y="0" z="${arm_length / 2.0}" color="yellow" />

Commit message: add plugin to control

File: my_robot_description/urdf/arm.xacro (robot description, xacro)
@@ -1,4 +1,4 @@
 <?xml version="1.0"?>
-<robot name="arm" xmlns:xacro="http://www.ros.org/wiki/xacro">
+<robot name="my_robot" xmlns:xacro="http://www.ros.org/wiki/xacro">
     <xacro:include filename="common_properties.xacro" />
     <xacro:property name="arm_base_length" value="0.1" />
@@ -13,5 +13,5 @@
                     <cylinder radius="${arm_radius}" length="${arm_length}" />
                 </geometry>
-                <origin xyz="${x} ${y} ${z}" />
+                <origin xyz="${x} ${y} ${z}" rpy="0 0 0"/>
                 <material name="${color}" />
             </visual>
@@ -20,5 +20,5 @@
                     <cylinder radius="${arm_radius}" length="${arm_length}" />
                 </geometry>
-                <origin xyz="${x} ${y} ${z}" />
+                <origin xyz="${x} ${y} ${z}" rpy="0 0 0"/>
             </collision>
             <xacro:cylinder_inertia m="0.3" r="${arm_radius}" h="${arm_length}"
@@ -26,5 +26,4 @@
         </link>
     </xacro:macro>
-    <link name="base_footprint" />
     <link name="arm_base_link">
         <visual>
@@ -32,5 +31,5 @@
                 <box size="${arm_base_length} ${arm_base_width} ${arm_base_height}" />
             </geometry>
-            <origin xyz="0 0 0" rpy="0 0 0"/>
+            <origin xyz="0 0 ${arm_base_height/2.0}" rpy="0 0 0"/>
             <material name="orange" />
         </visual>
@@ -39,22 +38,18 @@
                 <box size="${arm_base_length} ${arm_base_width} ${arm_base_height}" />
             </geometry>
+            <origin xyz="0 0 ${arm_base_height/2.0}" rpy="0 0 0"/>
         </collision>
-        <xacro:box_inertia m="0.5" x="${arm_base_length}" y="${arm_base_width}" z="${arm_base_height}"
-                           o_xyz="0 0 0" o_rpy="0 0 0" />
+        <xacro:box_inertia m="5.0" x="${arm_base_length}" y="${arm_base_width}" z="${arm_base_height}"
+                           o_xyz="0 0 ${arm_base_height/2.0}" o_rpy="0 0 0" />
     </link>
     <xacro:arms name="forearm" x="0" y="0" z="${arm_length / 2.0}" color="yellow" />
     <xacro:arms name="hand" x="0" y="0" z="${arm_length / 2.0}" color="orange" />
-    <joint name="arm_base_joint" type="fixed">
-        <parent link="base_footprint" />
-        <child link="arm_base_link" />
-        <origin xyz="0 0 0" rpy="0 0 0"/>
-    </joint>
     <joint name="base_forearm_joint" type="revolute">
         <parent link="arm_base_link" />
         <child link="forearm_link" />
         <axis xyz="0 1 0" />
-        <origin xyz="0 0 ${arm_base_height / 2.0}" rpy="0 0 0"/>
-        <limit lower="0" upper="${pi / 2.0}" effort="100" velocity="100" />
-        <dynamic friction="0.3" damping="0.3" />
+        <origin xyz="0 0 ${arm_base_height}" rpy="0 0 0"/>
+        <limit lower="0" upper="${pi/2}" effort="100" velocity="100" />
+        <dynamics friction="0.3" damping="0.3" />
     </joint>
     <joint name="forearm_hand_joint" type="revolute">
@@ -63,6 +58,7 @@
         <axis xyz="0 1 0" />
         <origin xyz="0 0 ${arm_length}" rpy="0 0 0"/>
-        <limit lower="0" upper="${pi / 2.0}" effort="100" velocity="100" />
-        <dynamic friction="0.3" damping="0.3" />
+        <limit lower="0" upper="${pi/2}" effort="100" velocity="100" />
+        <dynamics friction="0.3" damping="0.3" />
     </joint>
+    <xacro:include filename="arm_gazebo.xacro" />
 </robot>

Commit message: combine arm with cart

File: my_robot_description/urdf/arm.xacro (robot description, xacro)
@@ -1,5 +1,4 @@
 <?xml version="1.0"?>
-<robot name="my_robot" xmlns:xacro="http://www.ros.org/wiki/xacro">
-    <xacro:include filename="common_properties.xacro" />
+<robot xmlns:xacro="http://www.ros.org/wiki/xacro">
     <xacro:property name="arm_base_length" value="0.1" />
     <xacro:property name="arm_base_width" value="0.1" />
@@ -40,5 +39,5 @@
             <origin xyz="0 0 ${arm_base_height/2.0}" rpy="0 0 0"/>
         </collision>
-        <xacro:box_inertia m="5.0" x="${arm_base_length}" y="${arm_base_width}" z="${arm_base_height}"
+        <xacro:box_inertia m="0.5" x="${arm_base_length}" y="${arm_base_width}" z="${arm_base_height}"
                            o_xyz="0 0 ${arm_base_height/2.0}" o_rpy="0 0 0" />
     </link>

File: my_robot_description/urdf/arm_robot.xacro (robot description, xacro)
@@ -3,6 +3,3 @@
     <xacro:include filename="common_properties.xacro" />
     <xacro:include filename="arm.xacro" />
-    <xacro:include filename="mobile_base.xacro" />
-    <xacro:include filename="mobile_base_gazebo.xacro" />
-    <xacro:include filename="camera.xacro" />
 </robot>

File: my_robot_description/urdf/mobile_base.xacro (robot description, xacro)
@@ -82,3 +82,8 @@
         <origin xyz="0 0 ${wheel_radius}" />
     </joint>
+    <joint name="base_arm" type="fixed">
+        <parent link="base_link" />
+        <child link="arm_base_link" />
+        <origin xyz="${base_length / 4} 0 ${base_height}" />
+    </joint>
 </robot>
