Commit message: ros_control finished

File: my_robot_description/urdf/mobile_base.xacro (robot description, xacro)
@@ -82,8 +82,8 @@
         <origin xyz="0 0 ${wheel_radius}" />
     </joint>
-    <joint name="base_arm" type="fixed">
+    <!-- <joint name="base_arm" type="fixed">
         <parent link="base_link" />
         <child link="arm_base_link" />
         <origin xyz="${base_length / 4} 0 ${base_height}" />
-    </joint>
+    </joint> -->
 </robot>

File: my_robot_description/urdf/my_robot.urdf.xacro (robot description, xacro)
@@ -2,8 +2,8 @@
 <robot name="my_robot" xmlns:xacro="http://www.ros.org/wiki/xacro">
     <xacro:include filename="common_properties.xacro" />
-    <xacro:include filename="arm.xacro" />
+    <!-- <xacro:include filename="arm.xacro" /> -->
     <xacro:include filename="mobile_base.xacro" />
-    <xacro:include filename="mobile_base_gazebo.xacro" />
-    <!-- <xacro:include filename="ros2_control.xacro" /> -->
+    <!-- <xacro:include filename="mobile_base_gazebo.xacro" /> -->
+    <xacro:include filename="ros2_control.xacro" />
     <xacro:include filename="camera.xacro" />
 </robot>

File: my_robot_description/urdf/ros2_control.xacro (robot description, xacro)
@@ -24,5 +24,5 @@
     <gazebo>
         <plugin filename="libgz_ros2_control-system.so" name="gz_ros2_control::GazeboSimROS2ControlPlugin">
-            <!-- <parameters>$(find my_robot_bringup)/config/ros_controller.yaml</parameters> -->
+            <parameters>$(find my_robot_bringup)/config/ros_controller.yaml</parameters>
         </plugin>
     </gazebo>
